File: PCBs/reciever_ckt/reciever_ckt.kicad_sch (KiCad schematic)
At the start: 8 parts, among them J1 left, J2 right, J3 MQ3, J4 Button, J5 Battery, U1 LM7805_TO220

Commit message: Reciever Schematic Uploaded
Parts:
- added J4: Motor/Rear Wheel, Connector_JST:JST_EH_B2B-EH-A_1x02_P2.50mm_Vertical, symbol Connector_Generic:Conn_01x02
- added U2: L293D, Package_DIP:DIP-16_W7.62mm, symbol Driver_Motor:L293D
- J3: value MQ3 -> LCD/I2C
- J4: value Button -> Motor/Front wheel
Connections:
- net 3V: no longer J3.3 (Pin_3)
- net A0: no longer J3.2 (Pin_2)
- net D1: now also J3.1 (Pin_1)
- net D2: now also J3.2 (Pin_2)
- net D4: now also U2.2 (1A), U2.7 (2A); no longer J4.1 (Pin_1)
- net D7: no longer J3.1 (Pin_1)
- net GND: now also J4.2 (Pin_2), U2.12 (GND), U2.13 (GND), U2.4 (GND), U2.5 (GND)
- net VIN: now also J3.3 (Pin_3), U2.16 (VCC1), U2.8 (VCC2)
- new net 1Y: J4.1 (Pin_1), U2.3 (1Y)
- new net 2Y: J4.1 (Pin_1), U2.6 (2Y)
Other:
- note added: "Motor Driver L293D"
