File: PCBs/transmitter_ckt/transmitter_ckt.kicad_pcb (KiCad board)
At the start: 2 copper layers, 8 parts, among them J1 left, J2 right, J3 MQ3, J4 Button, J5 Battery, U1 LM7805_TO220

Commit message: Reciever Schematic Uploaded
Other:
- board text added: "ESP 8266"
Changed lines of the file:
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@@
     )
+  )
+  (gr_text "ESP 8266\n" (at 124.46 91.44) (layer "B.Cu")
+    (effects (font (size 1.5 1.5) (thickness 0.3) bold) (justify left bottom))
   )
   (gr_text "USB\n" (at 129.54 114.3) (layer "B.Cu")
